Commit message: Ship Nav2 on Gazebo AMR: fix /odom, map+AMCL bringup, CLI --nav2.
Add OdometryWithCovariance bridge and base_footprint, indoor occupancy map,
sim_amr_nav2.launch.py, agenticros up sim-amr --nav2 (CLI 0.5.3), navigate
smoke script, and docs/roadmap updates. MoveIt2 on sim-arm remains deferred.

Co-authored-by: Cursor <cursoragent@cursor.com>

File: ros2_ws/src/agenticros_sim/urdf/agenticros_amr.urdf.xacro (robot description, xacro)
@@ -16,4 +16,12 @@
 -->
 <robot name="agenticros_amr" xmlns:xacro="http://www.ros.org/wiki/xacro">
+  <!-- ===================== base_footprint (Nav2 / costmap convention) ===================== -->
+  <link name="base_footprint"/>
+  <joint name="base_footprint_joint" type="fixed">
+    <parent link="base_footprint"/>
+    <child link="base_link"/>
+    <!-- base_link visual origin is chassis center ~0.10 m above ground -->
+    <origin xyz="0 0 0.10" rpy="0 0 0"/>
+  </joint>
   <!-- ===================== base_link ===================== -->
   <link name="base_link">
